File: 555_Timer_Clock.kicad_pcb (KiCad board)
At the start: 2 copper layers, 39 x 25 mm, 13 parts, among them J2 CLK_Out, U1 ICM7555xB

Commit message: Edited PCB Design
Parts:
- added G***: LOGO, Special_Footprints:rawrOwO, F.Cu at (105.7, 63.3)
- added J1: +5V, my_footprints:Terminal_Block_5mm, F.Cu at (102.2, 72.2)
- added SW1: Trigger, my_footprints:slide_switch_2.54mm, F.Cu at (123.6, 81.2)
- added SW2: RST, my_footprints:tact_switch_5mm, F.Cu at (112.0, 81.3)
Routing:
- net GND: track 0.00 -> 81.8 mm, vias 0 -> 2
- net /Trigger: track 0.00 -> 37.6 mm
- net /+5V: track 0.00 -> 35.8 mm
- net /CLK_Out: track 0.00 -> 25.0 mm, vias 0 -> 1
- net /RST: track 0.00 -> 18.9 mm
- net Net-(U1-DISCH): track 0.00 -> 13.4 mm
- net Net-(D1-K): track 0.00 -> 9.22 mm
- net Net-(U1-CONT): track 0.00 -> 7.46 mm
